File: docs/designs/embedded-systems-drone.kicad_sch (KiCad schematic)
At the start: 20 parts, among them M1 Motor_DC, M2 Motor_DC, Q1 MMFTN3402, Q2 MMFTN3402, Q3 MMFTN3402, Q4 MMFTN3402, U1 ESP32-CAM

Commit message: Updated drone schematic. Moved designs folder into docs.
Parts:
- added BT2: 3.7V, symbol Device:Battery
Connections:
- net at BT1.1 (+), D1.1 (K), D2.1 (K)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: no longer U2. (GND)
- net at Q3.2, R3.2: now also U1.P$16 (GPIO4); no longer U1.P$13 (GPIO15)
- net at Q4.2, R4.2: now also U1.P$3 (GPIO3); no longer U1.P$14 (GPIO14)
- net at U1.P$15 (GPIO2): no longer U3. (INT)
- net at U3. (INT): no longer U1.P$16 (GPIO4)
- net at U1.P$4 (3V3/5V): no longer U3. (INT)
- net at U1.P$8 (3V3): now also U3. (INT)
- net at BT1.2 (-), Q1.3, Q2.3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: now also BT2.2 (-)
- new net: U1.P$13 (GPIO15), U3. (INT)
- new net: U1.P$14 (GPIO14), U3. (INT)
- new net: BT2.1 (+), U2. (GND)
Other:
- moved on the sheet: U2
